File: Kicad_design_files/LED_ARRAY.sch (KiCad schematic (older format))
At the start: 13 parts, among them U1 LT3474

Commit message: almost done with layout
Connections:
- net GND: now also D3.3 (thermal_isloated), D4.3 (thermal_isloated), D5.3 (thermal_isloated)
Changed lines of the file:
@@
 LIBS:valves
 LIBS:chroma_spotlight
+LIBS:chromatic_spotlight-cache
 EELAYER 27 0
 EELAYER END
@@
 Sheet 2 3
 Title ""
-Date "14 jan 2014"
+Date "15 jan 2014"
 Rev ""
 Comp ""
@@
 P 5150 3450
 AR Path="/52D1CCA6/52D1CE30" Ref="#PWR013"  Part="1"
-AR Path="/52D1E869/52D1CE30" Ref="#PWR019"  Part="1"
-F 0 "#PWR013" H 5150 3450 30  0001 C CNN
+AR Path="/52D1E869/52D1CE30" Ref="#PWR022"  Part="1"
+F 0 "#PWR022" H 5150 3450 30  0001 C CNN
 F 1 "GND" H 5150 3380 30  0001 C CNN
 F 2 "" H 5150 3450 60  0000 C CNN
@@
 P 5150 1950
 AR Path="/52D1CCA6/52D1CE38" Ref="#PWR014"  Part="1"
-AR Path="/52D1E869/52D1CE38" Ref="#PWR020"  Part="1"
-F 0 "#PWR014" H 5150 1900 20  0001 C CNN
+AR Path="/52D1E869/52D1CE38" Ref="#PWR023"  Part="1"
+F 0 "#PWR023" H 5150 1900 20  0001 C CNN
 F 1 "+12V" H 5150 2050 30  0000 C CNN
 F 2 "" H 5150 1950 60  0000 C CNN
@@
 P 4100 3150
 AR Path="/52D1CCA6/52D1CE83" Ref="#PWR015"  Part="1"
-AR Path="/52D1E869/52D1CE83" Ref="#PWR021"  Part="1"
-F 0 "#PWR015" H 4100 3150 30  0001 C CNN
+AR Path="/52D1E869/52D1CE83" Ref="#PWR024"  Part="1"
+F 0 "#PWR024" H 4100 3150 30  0001 C CNN
 F 1 "GND" H 4100 3080 30  0001 C CNN
 F 2 "" H 4100 3150 60  0000 C CNN
@@
 P 7150 2650
 AR Path="/52D1CCA6/52D1CEBB" Ref="#PWR016"  Part="1"
-AR Path="/52D1E869/52D1CEBB" Ref="#PWR022"  Part="1"
-F 0 "#PWR016" H 7150 2650 30  0001 C CNN
+AR Path="/52D1E869/52D1CEBB" Ref="#PWR025"  Part="1"
+F 0 "#PWR025" H 7150 2650 30  0001 C CNN
 F 1 "GND" H 7150 2580 30  0001 C CNN
 F 2 "" H 7150 2650 60  0000 C CNN
@@
 P 6850 3300
 AR Path="/52D1CCA6/52D1CEC2" Ref="#PWR017"  Part="1"
-AR Path="/52D1E869/52D1CEC2" Ref="#PWR023"  Part="1"
-F 0 "#PWR017" H 6850 3300 30  0001 C CNN
+AR Path="/52D1E869/52D1CEC2" Ref="#PWR026"  Part="1"
+F 0 "#PWR026" H 6850 3300 30  0001 C CNN
 F 1 "GND" H 6850 3230 30  0001 C CNN
 F 2 "" H 6850 3300 60  0000 C CNN
@@
 P 4400 2400
 AR Path="/52D1CCA6/52D1CED6" Ref="#PWR018"  Part="1"
-AR Path="/52D1E869/52D1CED6" Ref="#PWR024"  Part="1"
-F 0 "#PWR018" H 4400 2400 30  0001 C CNN
+AR Path="/52D1E869/52D1CED6" Ref="#PWR027"  Part="1"
+F 0 "#PWR027" H 4400 2400 30  0001 C CNN
 F 1 "GND" H 4400 2330 30  0001 C CNN
 F 2 "" H 4400 2400 60  0000 C CNN
@@
 Wire Wire Line
 	6500 3900 6550 3900
+$Comp
+L GND #PWR028
+U 1 1 52D714DE
+P 6600 2850
+AR Path="/52D1E869/52D714DE" Ref="#PWR028"  Part="1"
+AR Path="/52D1CCA6/52D714DE" Ref="#PWR019"  Part="1"
+F 0 "#PWR028" H 6600 2850 30  0001 C CNN
+F 1 "GND" H 6600 2780 30  0001 C CNN
+F 2 "" H 6600 2850 60  0000 C CNN
+F 3 "" H 6600 2850 60  0000 C CNN
+	1    6600 2850
+	1    0    0    -1
+$EndComp
+Wire Wire Line
+	6550 2800 6600 2800
+Wire Wire Line
+	6600 2800 6600 2850
+$Comp
+L GND #PWR029
+U 1 1 52D71522
+P 6600 3300
+AR Path="/52D1E869/52D71522" Ref="#PWR029"  Part="1"
+AR Path="/52D1CCA6/52D71522" Ref="#PWR020"  Part="1"
+F 0 "#PWR029" H 6600 3300 30  0001 C CNN
+F 1 "GND" H 6600 3230 30  0001 C CNN
+F 2 "" H 6600 3300 60  0000 C CNN
+F 3 "" H 6600 3300 60  0000 C CNN
+	1    6600 3300
+	1    0    0    -1
+$EndComp
+Wire Wire Line
+	6550 3250 6600 3250
+Wire Wire Line
+	6600 3250 6600 3300
+$Comp
+L GND #PWR030
+U 1 1 52D7152A
+P 6600 3750
+AR Path="/52D1E869/52D7152A" Ref="#PWR030"  Part="1"
+AR Path="/52D1CCA6/52D7152A" Ref="#PWR021"  Part="1"
+F 0 "#PWR030" H 6600 3750 30  0001 C CNN
+F 1 "GND" H 6600 3680 30  0001 C CNN
+F 2 "" H 6600 3750 60  0000 C CNN
+F 3 "" H 6600 3750 60  0000 C CNN
+	1    6600 3750
+	1    0    0    -1
+$EndComp
+Wire Wire Line
+	6550 3700 6600 3700
+Wire Wire Line
+	6600 3700 6600 3750
 $EndSCHEMATC

Commit message: added numerous improvements
Connections:
- net link_4: now reaches D3.1 (A), U1.3 (LED)
- net link_1: now reaches D3.2 (K), D4.1 (A)
- net link_2: now reaches D4.2 (K), D5.1 (A)
Changed lines of the file:
@@
 Sheet 2 3
 Title ""
-Date "15 jan 2014"
+Date "16 jan 2014"
 Rev ""
 Comp ""
@@
 AR Path="/52D1CCA6/52D1CE30" Ref="#PWR013"  Part="1"
 AR Path="/52D1E869/52D1CE30" Ref="#PWR022"  Part="1"
-F 0 "#PWR022" H 5150 3450 30  0001 C CNN
+F 0 "#PWR013" H 5150 3450 30  0001 C CNN
 F 1 "GND" H 5150 3380 30  0001 C CNN
 F 2 "" H 5150 3450 60  0000 C CNN
@@
 AR Path="/52D1CCA6/52D1CE38" Ref="#PWR014"  Part="1"
 AR Path="/52D1E869/52D1CE38" Ref="#PWR023"  Part="1"
-F 0 "#PWR023" H 5150 1900 20  0001 C CNN
+F 0 "#PWR014" H 5150 1900 20  0001 C CNN
 F 1 "+12V" H 5150 2050 30  0000 C CNN
 F 2 "" H 5150 1950 60  0000 C CNN
@@
 AR Path="/52D1CCA6/52D1CE83" Ref="#PWR015"  Part="1"
 AR Path="/52D1E869/52D1CE83" Ref="#PWR024"  Part="1"
-F 0 "#PWR024" H 4100 3150 30  0001 C CNN
+F 0 "#PWR015" H 4100 3150 30  0001 C CNN
 F 1 "GND" H 4100 3080 30  0001 C CNN
 F 2 "" H 4100 3150 60  0000 C CNN
@@
 AR Path="/52D1CCA6/52D1CEBB" Ref="#PWR016"  Part="1"
 AR Path="/52D1E869/52D1CEBB" Ref="#PWR025"  Part="1"
-F 0 "#PWR025" H 7150 2650 30  0001 C CNN
+F 0 "#PWR016" H 7150 2650 30  0001 C CNN
 F 1 "GND" H 7150 2580 30  0001 C CNN
 F 2 "" H 7150 2650 60  0000 C CNN
@@
 AR Path="/52D1CCA6/52D1CEC2" Ref="#PWR017"  Part="1"
 AR Path="/52D1E869/52D1CEC2" Ref="#PWR026"  Part="1"
-F 0 "#PWR026" H 6850 3300 30  0001 C CNN
+F 0 "#PWR017" H 6850 3300 30  0001 C CNN
 F 1 "GND" H 6850 3230 30  0001 C CNN
 F 2 "" H 6850 3300 60  0000 C CNN
@@
 AR Path="/52D1CCA6/52D1CED6" Ref="#PWR018"  Part="1"
 AR Path="/52D1E869/52D1CED6" Ref="#PWR027"  Part="1"
-F 0 "#PWR027" H 4400 2400 30  0001 C CNN
+F 0 "#PWR018" H 4400 2400 30  0001 C CNN
 F 1 "GND" H 4400 2330 30  0001 C CNN
 F 2 "" H 4400 2400 60  0000 C CNN
@@
 Text HLabel 5100 2200 0    60   Input ~ 0
 SHDN
-Text HLabel 6550 3900 2    60   UnSpc ~ 0
+Text HLabel 6850 3900 2    60   UnSpc ~ 0
 LED_CATHODE
 Text HLabel 5100 2700 0    60   Input ~ 0
@@
 	5100 2700 5150 2700
 Wire Wire Line
-	6500 3900 6550 3900
+	6500 3900 6850 3900
 $Comp
 L GND #PWR028
@@
 AR Path="/52D1E869/52D714DE" Ref="#PWR028"  Part="1"
 AR Path="/52D1CCA6/52D714DE" Ref="#PWR019"  Part="1"
-F 0 "#PWR028" H 6600 2850 30  0001 C CNN
+F 0 "#PWR019" H 6600 2850 30  0001 C CNN
 F 1 "GND" H 6600 2780 30  0001 C CNN
 F 2 "" H 6600 2850 60  0000 C CNN
@@
 AR Path="/52D1E869/52D71522" Ref="#PWR029"  Part="1"
 AR Path="/52D1CCA6/52D71522" Ref="#PWR020"  Part="1"
-F 0 "#PWR029" H 6600 3300 30  0001 C CNN
+F 0 "#PWR020" H 6600 3300 30  0001 C CNN
 F 1 "GND" H 6600 3230 30  0001 C CNN
 F 2 "" H 6600 3300 60  0000 C CNN
@@
 AR Path="/52D1E869/52D7152A" Ref="#PWR030"  Part="1"
 AR Path="/52D1CCA6/52D7152A" Ref="#PWR021"  Part="1"
-F 0 "#PWR030" H 6600 3750 30  0001 C CNN
+F 0 "#PWR021" H 6600 3750 30  0001 C CNN
 F 1 "GND" H 6600 3680 30  0001 C CNN
 F 2 "" H 6600 3750 60  0000 C CNN
@@
 Wire Wire Line
 	6600 3700 6600 3750
+Text Label 6500 3000 0    60   ~ 0
+link_1
+Text Label 6500 3450 0    60   ~ 0
+link_2
+Text Label 6500 3900 0    60   ~ 0
+link_3
+Text Label 6500 2550 0    60   ~ 0
+link_4
 $EndSCHEMATC
