File: Kicad_design_files/chromatic_spotlight.sch (KiCad schematic (older format))
At the start: 9 parts, among them CON1 POWER_CONN, P1 CONN_6, Q1 MOSFET_N, Q2 MOSFET_N, SW1 SLIDE 1PDT

Commit message: almost done with layout
Connections:
- net +12V: now also SW1.1; no longer SW1.3
- net GND: now also SW1.3; no longer SW1.1
Changed lines of the file:
@@
 LIBS:valves
 LIBS:chroma_spotlight
+LIBS:chromatic_spotlight-cache
 EELAYER 27 0
 EELAYER END
@@
 Sheet 1 3
 Title ""
-Date "14 jan 2014"
+Date "15 jan 2014"
 Rev ""
 Comp ""
@@
 F 3 "~" H 1700 2050 60  0000 C CNN
 	1    1700 2050
-	-1   0    0    1
+	-1   0    0    -1
 $EndComp
 $Comp

Commit message: added numerous improvements
Parts:
- added P?: CONN_1, ~, symbol CONN_1
Connections:
- net GND: now also P?.1
Changed lines of the file:
@@
 Sheet 1 3
 Title ""
-Date "15 jan 2014"
+Date "16 jan 2014"
 Rev ""
 Comp ""
@@
 0.04375V - 1.25V MAX
 NoConn ~ 1300 3700
+$Comp
+L CONN_1 P?
+U 1 1 52D7555B
+P 3450 3800
+F 0 "P?" H 3530 3800 40  0000 L CNN
+F 1 "CONN_1" H 3450 3855 30  0001 C CNN
+F 2 "~" H 3450 3800 60  0000 C CNN
+F 3 "~" H 3450 3800 60  0000 C CNN
+	1    3450 3800
+	-1   0    0    1
+$EndComp
+$Comp
+L GND #PWR?
+U 1 1 52D755C2
+P 3650 3850
+F 0 "#PWR?" H 3650 3850 30  0001 C CNN
+F 1 "GND" H 3650 3780 30  0001 C CNN
+F 2 "" H 3650 3850 60  0000 C CNN
+F 3 "" H 3650 3850 60  0000 C CNN
+	1    3650 3850
+	1    0    0    -1
+$EndComp
+Wire Wire Line
+	3600 3800 3650 3800
+Wire Wire Line
+	3650 3800 3650 3850
 $EndSCHEMATC

Commit message: going home for the night
Other:
- note added: "psuedo part for camera hole"
Changed lines of the file:
@@
 Wire Wire Line
 	3650 3800 3650 3850
+Text Notes 3050 3700 0    60   ~ 0
+psuedo part for camera hole
 $EndSCHEMATC
